File: LT3045_breakout.kicad_pcb (KiCad board)
At the start: 2 copper layers, 10.2 x 14.6 mm, 12 parts, among them J1 CONN_01X03, U1 LT3045EDD

Commit message: Added label '78xx' to the board Added .gitignore file
Other:
- board text added: "78xx"
Changed lines of the file:
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@@
     (area 104.477381 86.924999 130.022619 110.925001)
     (thickness 1.6)
-    (drawings 7)
+    (drawings 8)
     (tracks 129)
     (zones 0)
@@
     )
   )
+  (gr_text 78xx (at 121.3 91.9) (layer B.SilkS)
+    (effects (font (size 0.8 0.8) (thickness 0.2)) (justify mirror))
+  )
   (gr_text "by Patrick Baus" (at 118.1 98.25) (layer B.SilkS)
