File: LT3045_breakout.kicad_pcb (KiCad board)
At the start: 2 copper layers, 10.2 x 14.6 mm, 12 parts, among them J1 CONN_01X03, U1 LT3045EDD

Commit message: Added more descriptive text to the board
Other:
- board text added: "G"
- board text added: "I"
- board text added: "LT3042"
- board text added: "LT3045"
- board text added: "O"
- board text removed: "78xx"
Changed lines of the file:
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@@
     (area 104.477381 86.924999 130.022619 110.925001)
     (thickness 1.6)
-    (drawings 8)
+    (drawings 12)
     (tracks 129)
     (zones 0)
@@
     (34 B.Paste user)
     (35 F.Paste user)
-    (36 B.SilkS user hide)
+    (36 B.SilkS user)
     (37 F.SilkS user)
     (38 B.Mask user)
@@
     )
   )
-  (gr_text 78xx (at 121.3 91.9) (layer B.SilkS)
+  (gr_text G (at 116.8 98.8) (layer F.SilkS)
+    (effects (font (size 0.8 0.8) (thickness 0.2)))
+  )
+  (gr_text O (at 122.5 100.3) (layer F.SilkS)
+    (effects (font (size 0.8 0.8) (thickness 0.2)))
+  )
+  (gr_text I (at 113.9 100.2) (layer F.SilkS)
+    (effects (font (size 0.8 0.8) (thickness 0.2)))
+  )
+  (gr_text LT3045 (at 121.9 94.1 90) (layer B.SilkS)
     (effects (font (size 0.8 0.8) (thickness 0.2)) (justify mirror))
   )
+  (gr_text LT3042 (at 114.4 94.1 90) (layer B.SilkS)
+    (effects (font (size 0.8 0.8) (thickness 0.2)) (justify mirror))
+  )

Commit message: Removed PGFB pull resistor. We do not need that.
Parts:
- removed the R1 at (118.5, 98.4)
- renumbered R2 to R1, R3 to R2, R4 to R3, R5 to R4
Routing:
- net Net-(U1-Pad6): track 3.18 -> 0.00 mm

Commit message: Changed resistor values to outout 12V@500mA
Parts:
- R1: value 100k -> 121k
- R2: value 100k -> 300
Changed lines of the file:
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@@
       (effects (font (size 1 1) (thickness 0.15)))
     )
-    (fp_text value 100k (at 0 1.5 270) (layer F.Fab)
+    (fp_text value 121k (at 0 1.5 270) (layer F.Fab)
       (effects (font (size 1 1) (thickness 0.15)))
     )
@@
       (effects (font (size 1 1) (thickness 0.15)))
     )
-    (fp_text value 100k (at 0 1.5 180) (layer F.Fab)
+    (fp_text value 300 (at 0 1.5 180) (layer F.Fab)
       (effects (font (size 1 1) (thickness 0.15)))
     )

Commit message: Added text to denote Rlim and Rset Changed 3d model of the pin header
Other:
- board text added: "Rlim"
- board text added: "Rset"
Changed lines of the file:
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@@
     (area 104.477381 86.924999 130.022619 110.925001)
     (thickness 1.6)
-    (drawings 12)
+    (drawings 14)
     (tracks 124)
     (zones 0)
@@
       (net 5 /out))
     (model ${KISYS3DMOD}/Pin_Headers.3dshapes/Pin_Header_Angled_1x03_Pitch2.54mm.wrl
-      (at (xyz 0 -0.1 0))
-      (scale (xyz 1 1 1))
-      (rotate (xyz 0 0 90))
+      (at (xyz 0 0 0))
+      (scale (xyz 1 1 1))
+      (rotate (xyz 0 0 0))
     )
   )
@@
     )
   )
+  (gr_text Rlim (at 113.9 97.1 90) (layer F.SilkS)
+    (effects (font (size 0.8 0.8) (thickness 0.15)))
+  )
+  (gr_text Rset (at 122.4 96.2 90) (layer F.SilkS)
+    (effects (font (size 0.8 0.8) (thickness 0.15)))
+  )
   (gr_text G (at 116.8 98.8) (layer F.SilkS)
