File: LT3045_breakout.kicad_pcb (KiCad board)
At the start: 2 copper layers, 10.2 x 14.6 mm, 11 parts, among them J1 CONN_01X03, U1 LT3045EDD

Commit message: Updated libraries
Parts:
- R1: value 121k -> 120k
- R3: value 100k -> 200k
- R4: value 100k -> 5.6k
Connections:
- net IN2 renamed /in
